File: AccLoad/AccLoad.kicad_pcb (KiCad board)
At the start: 2 copper layers, 59.2 x 39.5 mm, 15 parts, among them J1 to MCU

Commit message: fixed error in PCB with voltmeter
Routing:
- net bat1+: track 55.8 -> 58.0 mm
Other:
- outline, holes or cut-outs redrawn
Changed lines of the file:
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@@
       (disableapertmacros false)
       (usegerberextensions false)
-      (usegerberattributes true)
-      (usegerberadvancedattributes true)
-      (creategerberjobfile true)
+      (usegerberattributes false)
+      (usegerberadvancedattributes false)
+      (creategerberjobfile false)
       (svguseinch false)
       (svgprecision 6)
-      (excludeedgelayer true)
+      (excludeedgelayer false)
       (plotframeref false)
       (viasonmask false)
@@
       (plotinvisibletext false)
       (sketchpadsonfab false)
-      (subtractmaskfromsilk false)
-      (outputformat 4)
+      (subtractmaskfromsilk true)
+      (outputformat 1)
       (mirror false)
       (drillshape 0)
       (scaleselection 1)
-      (outputdirectory "")
+      (outputdirectory "export/")
     )
   )
@@
   (gr_line (start 149.757 88.942) (end 151.057 88.942) (layer "Dwgs.User") (width 0.25))
   (gr_line locked (start 163.957 107.442) (end 163.957 67.942) (layer "Edge.Cuts") (width 0.25))
-  (gr_arc locked (start 132.957 72.242) (mid 133.044868 72.029868) (end 133.257 71.942) (layer "Edge.Cuts") (width 0.25))
-  (gr_arc locked (start 155.657 71.942) (mid 155.869132 72.029868) (end 155.957 72.242) (layer "Edge.Cuts") (width 0.25))
-  (gr_line locked (start 155.657 71.942) (end 133.257 71.942) (layer "Edge.Cuts") (width 0.25))
-  (gr_line locked (start 132.957 72.242) (end 132.957 82.142) (layer "Edge.Cuts") (width 0.25))
   (gr_circle locked (center 157.457 77.192) (end 158.357 77.192) (layer "Edge.Cuts") (width 0.25) (fill none))
   (gr_line locked (start 163.957 67.942) (end 104.757 67.942) (layer "Edge.Cuts") (width 0.25))
   (gr_circle locked (center 131.457 77.192) (end 132.357 77.192) (layer "Edge.Cuts") (width 0.25) (fill none))
-  (gr_arc locked (start 133.257 82.442) (mid 133.044868 82.354132) (end 132.957 82.142) (layer "Edge.Cuts") (width 0.25))
   (gr_line locked (start 104.757 67.942) (end 104.757 107.442) (layer "Edge.Cuts") (width 0.25))
-  (gr_arc locked (start 155.957 82.142) (mid 155.869132 82.354132) (end 155.657 82.442) (layer "Edge.Cuts") (width 0.25))
   (gr_line locked (start 104.757 107.442) (end 163.957 107.442) (layer "Edge.Cuts") (width 0.25))
-  (gr_line locked (start 155.957 82.142) (end 155.957 72.242) (layer "Edge.Cuts") (width 0.25))
-  (gr_line locked (start 133.257 82.442) (end 155.657 82.442) (layer "Edge.Cuts") (width 0.25))
+  (gr_rect locked (start 132.958601 71.943907) (end 155.955736 82.447233) (layer "Edge.Cuts") (width 0.1) (fill solid))
   (gr_text "-" (at 154.922 83.944) (layer "B.SilkS")
     (effects (font (size 1 1) (thickness 0.15)))
@@
   (segment (start 152.636 85.595) (end 152.636 83.817) (width 0.5) (layer "F.Cu") (net 3))
   (via (at 152.636 85.595) (size 0.8) (drill 0.4) (layers "F.Cu" "B.Cu") (net 3))
+  (segment (start 152.636 86.865) (end 150.477 86.865) (width 0.5) (layer "B.Cu") (net 3))
   (segment (start 152.636 86.865) (end 152.636 85.595) (width 0.5) (layer "B.Cu") (net 3))
   (segment (start 154.956102 99.242699) (end 154.922 99.208597) (width 0.5) (layer "F.Cu") (net 4))
